Commit message: ros

File: src/robot_description/urdf/m2wr.xacro (robot description, xacro)
@@ -75,6 +75,6 @@
   </joint>
   <xacro:link_wheel name="link_right_wheel" />
-  <xacro:joint_wheel name="joint_right_wheel" child="link_right_wheel" origin_xyz="-0.05 0.20 0" />
+  <xacro:joint_wheel name="joint_right_wheel" child="link_right_wheel" origin_xyz="-0.05 -0.20 0" />
   <xacro:link_wheel name="link_left_wheel" />
-  <xacro:joint_wheel name="joint_left_wheel" child="link_left_wheel" origin_xyz="-0.05 -0.20 0" />
+  <xacro:joint_wheel name="joint_left_wheel" child="link_left_wheel" origin_xyz="-0.05 0.20 0" />
 </robot>

File: src/robot_description/urdf/robot.urdf (robot description, URDF)
Before this commit: robot my_robot, 8 links, 7 joints
Links:
- link chassis: geometry visual box size=0.60 0.4 0.334
Joints:
- joint fake_joint: origin xyz=0.0 0.0 0.22 -> xyz=0.0 0.0 0.24
